File: schematics/window_control/full_schema.sch (EAGLE design)
At the start: 72 parts, among them J1 MTR-SERVO-FS5103B, J10 USBASP_PIN, J2 J2, J3 J2, J4 J2, J5 J2, J6 J2, J7 J2, J8 J2, J9 J2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

Commit message: full schema on atmega328 tested and worked
Parts:
- removed R26: 200K, my_devices:RD
- added R21: 10K, my_devices:R
- C10: value 0.1 uF -> 10 uF; device my_devices:C-1 -> my_devices:C
- C9: value 10 uF -> 0.1 uF; device my_devices:C -> my_devices:C-1
- R10: value 100 -> 200
- R11: value 10K -> 100
- R13: value 100 -> 10K
- R14: value 5 -> 100
- R15: value 3K -> 5
- R16: value 200K -> 3K
- R17: value 5K -> 10K
- R18: value 10K -> 3K; device my_devices:RD -> my_devices:R
- R20: value 10K -> 200K; device my_devices:R -> my_devices:RD
- R22: value 3K -> 200K
- R6: value 620 -> 5K; device my_devices:R -> my_devices:RD
- R8: value 20K -> 620; device my_devices:RD -> my_devices:R
- R9: value 200 -> 20K; device my_devices:R -> my_devices:RD
- U6: value ATMEGA328P -> LM317L; device my_devices:ATMEGA328P -> my_devices:VOLTAGE_REGULATOR
- U7: value LM317L -> LM358; device my_devices:VOLTAGE_REGULATOR -> my_devices:LM358
- U8: value GY-SGP30 -> ATMEGA328P; device my_devices:GY-SGP30 -> my_devices:ATMEGA328P
- U9: value LM358 -> GY-SGP30; device my_devices:LM358 -> my_devices:GY-SGP30
- renumbered BM2 to BM1, C12 to C11, C13 to C7, C15 to C8
Connections:
- net +5V_IF_EN: now also R11.P$2; no longer R10.P$2
- net 3V3: now also R12.P$1, R13.P$2; no longer R11.P$1, R12.P$2
- net ATMEGA_RESET: now also C9.P$2, R21.P$1, U8.PC6; no longer C10.P$2, R20.P$1, U6.PC6
- net ATMEGA_RXD: now also U8.PD1; no longer U6.PD1
- net ATMEGA_TXD: now also U8.PD0; no longer U6.PD0
- net GND: now also J3.PIN_1, R10.P$2, R16.P$1, R6.P1; no longer J9.PIN_1, R15.P$1, R17.P1, R9.P$2
- net HALL_OUT_INV: now also R13.P$1, R8.P$2; no longer R12.P$1, R7.P$2
- net I2C_SCL: now also U8.PC5, U9.SCL; no longer U6.PC5, U8.SCL
- net I2C_SDA: now also U8.PC4, U9.SDA; no longer U6.PC4, U8.SDA
- net N$1: now also R15.P$1; no longer R14.P$1
- net N$10: now also J4.PIN_2, J6.PIN_1; no longer J3.PIN_2, J4.PIN_1
- net N$11: now also J5.PIN_1; no longer J8.PIN_1
- net N$12: now also J5.PIN_2; no longer J8.PIN_2
- net N$13: now also R6.P3; no longer R17.P3
- net N$14: now also R18.P$2; no longer R22.P$2
- net N$15: now also R19.P$2, U7.A+; no longer R16.P$2, U9.A+
- net N$17: now also R17.P3, U6.GND; no longer R18.P3, U7.GND
- net N$18: now also R20.P1, U7.A_OUT; no longer R23.P1, U9.A_OUT
- net N$19: now also R23.P3, U7.B-; no longer R26.P3, U9.B-
- net N$2: now also R14.P$2; no longer R13.P$2
- net N$20: now also R22.P$1, U7.B+; no longer R19.P$1, U9.B+
- net N$21: now also R20.P3, U7.A-; no longer R23.P3, U9.A-
- net N$24: now also U8.PB3; no longer U6.PB3
- net N$25: now also U8.PB4; no longer U6.PB4
- net N$26: now also U8.PB5; no longer U6.PB5
- net N$28: now also R7.P$1; no longer R6.P$1
- net N$29: now also R8.P$1; no longer R7.P$1
- net N$35: now also R14.P$1; no longer R13.P$1
- net N$38: now also R10.P$1; no longer R9.P$1
- net N$39: now also D4.ANODE, R15.P$2; no longer D4.P$1, R14.P$2
- net N$47: now also R9.P3; no longer R8.P3
- net N$48: now also R9.P2; no longer R8.P2
- net N$49: now also R11.P$1, R9.P1; no longer R10.P$1, R8.P1
- net N$51: now also D4.CATHODE, R16.P$2; no longer D4.P$2, R15.P$2
- net N$9: now also J4.PIN_1, J6.PIN_2; no longer J3.PIN_1, J4.PIN_2
- net NOISE_LEVEL: now also R23.P2, U7.B_OUT, U8.PC1; no longer R26.P2, U6.PC1, U9.B_OUT
- net OUT: now also L3.P$1, R17.P2, U6.OUT; no longer L2.P$1, R18.P2, U7.OUT
- net OUTDOOR_+5V: now also J8.PIN_1, L2.P$1, R21.P$2, U8.AREF, U8.AVCC, U8.VCC, U9.VIN; no longer J5.PIN_1, L3.P$1, R20.P$2, U6.AREF, U6.AVCC, U6.VCC, U8.VIN
- net OUTDOOR_+5V_F: now also L2.P$2, R18.P$1, U6.IN, U7.VCC; no longer L3.P$2, R22.P$1, U7.IN, U9.VCC
- net OUTDOOR_DATA_OUT: now also J9.PIN_1, U8.PC3; no longer J6.PIN_1, U6.PC3
- net OUTDOOR_GND: now also C10.PIN_GND, C9.P$1, J8.PIN_2, J9.PIN_2, R17.P1, U7.VEE, U8.GND1, U9.GND; no longer C10.P$1, C9.PIN_GND, J5.PIN_2, J6.PIN_2, R18.P1, U6.GND, U6.GND1, U9.VEE
- net OUTDOOR_MIDDLEPOINT: now also C10.PIN_PLUS, L3.P$2, R19.P$1, R20.P2, R22.P$2, R23.P1; no longer C9.PIN_PLUS, L2.P$2, R16.P$1, R19.P$2, R23.P2, R26.P1
- net OUTDOOR_SIGNAL: now also J3.PIN_2, R6.P2; no longer J9.PIN_2, R17.P2
- net SERVO_ENABLE_INV: now also R7.P$2; no longer R6.P$2
- net SW_IS_ON_INV: now also R12.P$2; no longer R11.P$2
Other:
- moved on the sheet: J3, J4, J5, J6, J8, J9, L2, L3, R10, R11, R12, R13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

Commit message: Start boards preparing - actualized new element dimentions
Parts:
- L1: value 1000 uH -> RLB0914-102KL, 1000 uH
- L2, L3: value 560 uH -> EC24-561K, 560 uH; device my_devices:L -> my_devices:LL-EC24
- R20, R23: device my_devices:RD -> my_devices:RD3296-Z
- U5: value BMP280 / 5V -> BMP280 5V module
Changed lines of the file:
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@@
 <part name="TS2" library="my_devices" deviceset="TOUCH_SENSOR" device=""/>
 <part name="R21" library="my_devices" deviceset="R" device="" value="10K"/>
-<part name="U5" library="my_devices" deviceset="BME280" device="" value="BMP280 / 5V"/>
+<part name="U5" library="my_devices" deviceset="BME280" device="" value="BMP280 5V module"/>
 <part name="U9" library="my_devices" deviceset="GY-SGP30" device=""/>
 <part name="B1" library="my_devices" deviceset="HALL_SENSOR" device="" value="A3144"/>
@@
 <part name="R8" library="my_devices" deviceset="R" device="" value="620"/>
 <part name="D4" library="my_devices" deviceset="D_SCHOTTKY" device="" value="BAT41"/>
-<part name="L1" library="my_devices" deviceset="L" device="" value="1000 uH"/>
+<part name="L1" library="my_devices" deviceset="L" device="" value="RLB0914-102KL, 1000 uH"/>
 <part name="Q3" library="my_devices" deviceset="TRANSISTOR_PNP" device="" value="2N3906BU"/>
 <part name="Q5" library="my_devices" deviceset="MOSFET_N" device="" value="STP14NM50N"/>
@@
 <part name="R18" library="my_devices" deviceset="R" device="" value="3K"/>
 <part name="C8" library="my_devices" deviceset="C-1" device="" value="0.1 uF"/>
-<part name="R20" library="my_devices" deviceset="RD" device="" value="200K"/>
-<part name="R23" library="my_devices" deviceset="RD" device="" value="200K"/>
+<part name="R20" library="my_devices" deviceset="RD" device="3296-Z" value="200K"/>
+<part name="R23" library="my_devices" deviceset="RD" device="3296-Z" value="200K"/>
 <part name="U6" library="my_devices" deviceset="VOLTAGE_REGULATOR" device="" value="LM317L"/>
-<part name="L3" library="my_devices" deviceset="L" device="" value="560 uH"/>
+<part name="L3" library="my_devices" deviceset="L" device="L-EC24" value="EC24-561K, 560 uH"/>
 <part name="C10" library="my_devices" deviceset="C" device="" value="10 uF"/>
 <part name="R19" library="my_devices" deviceset="R" device="" value="200K"/>
@@
 <part name="C11" library="my_devices" deviceset="C-1" device="" value="0.1 uF"/>
 <part name="R22" library="my_devices" deviceset="R" device="" value="200K"/>
-<part name="L2" library="my_devices" deviceset="L" device="" value="560 uH"/>
+<part name="L2" library="my_devices" deviceset="L" device="L-EC24" value="EC24-561K, 560 uH"/>
 <part name="C7" library="my_devices" deviceset="C" device="" value="10 uF"/>
 <part name="U8" library="my_devices" deviceset="ATMEGA328P" device=""/>

Commit message: Touch sensor are unstable. I made a decision to replace it by normally-open buttons
Parts:
- removed TS1, TS2, TS3: TOUCH_SENSOR, my_devices:TOUCH_SENSOR
- added SB1: SB-NC, my_devices:SB-NC
- added SB2, SB3, SB4: SB-NO, my_devices:SB-NO
- SW1: value SWITCH -> MRS-101-2C3-B
Connections:
- new net N$16: J2.PIN_2, SB1.P$2
- net +5V: now also SB1.P$1; no longer J2.PIN_2
- net GND: now also SB2.P$2, SB3.P$2, SB4.P$2
- net GPIO_TS_WINDOW_AUTO: now also SB4.P$1; no longer TS3.P$1
- net GPIO_TS_WINDOW_CLOSE: now also SB3.P$1; no longer TS2.P$1
- net GPIO_TS_WINDOW_OPEN: now also SB2.P$1; no longer TS1.P$1
Changed lines of the file:
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@@
 <part name="U1" library="my_devices" deviceset="ESP32" device=""/>
 <part name="GND2" library="supply1" library_urn="urn:adsk.eagle:library:371" deviceset="GND" device=""/>
-<part name="TS1" library="my_devices" deviceset="TOUCH_SENSOR" device=""/>
-<part name="TS2" library="my_devices" deviceset="TOUCH_SENSOR" device=""/>
 <part name="R21" library="my_devices" deviceset="R" device="" value="10K"/>
 <part name="U5" library="my_devices" deviceset="BME280" device="" value="BMP280 5V module"/>
@@
 <part name="J1" library="my_devices" deviceset="SERVO" device="" value="MTR-SERVO-FS5103B"/>
 <part name="GND3" library="supply1" library_urn="urn:adsk.eagle:library:371" deviceset="GND" device=""/>
-<part name="SW1" library="my_devices" deviceset="SWITCH" device=""/>
+<part name="SW1" library="my_devices" deviceset="SWITCH" device="" value="MRS-101-2C3-B"/>
 <part name="GND4" library="supply1" library_urn="urn:adsk.eagle:library:371" deviceset="GND" device=""/>
 <part name="U4" library="my_devices" deviceset="SN74LS32N" device=""/>
@@
 <part name="GND7" library="supply1" library_urn="urn:adsk.eagle:library:371" deviceset="GND" device=""/>
 <part name="R1" library="my_devices" deviceset="R" device="" value="620"/>
-<part name="TS3" library="my_devices" deviceset="TOUCH_SENSOR" device=""/>
 <part name="J2" library="my_devices" deviceset="J2" device=""/>
 <part name="J4" library="my_devices" deviceset="J2" device=""/>
@@
 <part name="C9" library="my_devices" deviceset="C-1" device="" value="0.1 uF"/>
 <part name="J10" library="my_devices" deviceset="USBASP_PIN" device=""/>
+<part name="SB1" library="my_devices" deviceset="SB-NC" device=""/>
+<part name="SB2" library="my_devices" deviceset="SB-NO" device=""/>
+<part name="SB3" library="my_devices" deviceset="SB-NO" device=""/>
+<part name="SB4" library="my_devices" deviceset="SB-NO" device=""/>
+<part name="GND9" library="supply1" library_urn="urn:adsk.eagle:library:371" deviceset="GND" device=""/>
 </parts>
 <sheets>
@@
 <attribute name="VALUE" x="-154.94" y="142.24" size="1.778" layer="96"/>
 </instance>
-<instance part="TS1" gate="G$1" x="-27.94" y="5.08" smashed="yes" grouprefs="OPEN-CLOSE">
-<attribute name="NAME" x="-33.02" y="10.16" size="1.778" layer="94"/>
-</instance>
-<instance part="TS2" gate="G$1" x="-27.94" y="-15.24" smashed="yes" grouprefs="OPEN-CLOSE">
-<attribute name="NAME" x="-33.02" y="-10.16" size="1.778" layer="94"/>
-</instance>
 <instance part="R21" gate="G$1" x="259.08" y="170.18" smashed="yes" rot="R90" grouprefs="ATMEGA32">
 <attribute name="NAME" x="256.54" y="163.83" size="1.778" layer="94" rot="R90"/>
@@
 <attribute name="VALUE" x="-222.25" y="44.45" size="1.778" layer="94"/>
 </instance>
-<instance part="TS3" gate="G$1" x="-27.94" y="-35.56" smashed="yes" grouprefs="OPEN-CLOSE">
-<attribute name="NAME" x="-33.02" y="-30.48" size="1.778" layer="94"/>
-</instance>
 <instance part="J2" gate="G$1" x="73.66" y="142.24" smashed="yes" rot="R180" grouprefs="INDOOR_TO_OUTDOOR_CABEL">
 <attribute name="NAME" x="76.2" y="140.335" size="1.778" layer="94" rot="R180"/>
@@
 <attribute name="NAME" x="330.835" y="112.395" size="0.8128" layer="94"/>
 <attribute name="VALUE" x="330.835" y="94.615" size="0.8128" layer="94"/>
+</instance>
+<instance part="SB1" gate="G$1" x="53.34" y="144.78" smashed="yes" grouprefs="INDOOR_TO_OUTDOOR_CABEL">
+<attribute name="NAME" x="48.26" y="142.24" size="1.778" layer="94"/>
+<attribute name="VALUE" x="48.26" y="139.7" size="1.778" layer="94"/>
+</instance>
+<instance part="SB2" gate="G$1" x="-25.4" y="5.08" smashed="yes" grouprefs="OPEN-CLOSE">
+<attribute name="NAME" x="-30.48" y="2.54" size="1.778" layer="94"/>
+<attribute name="VALUE" x="-30.48" y="0" size="1.778" layer="94"/>
+</instance>
+<instance part="SB3" gate="G$1" x="-25.4" y="-15.24" smashed="yes" grouprefs="OPEN-CLOSE">
+<attribute name="NAME" x="-30.48" y="-17.78" size="1.778" layer="94"/>
+<attribute name="VALUE" x="-30.48" y="-20.32" size="1.778" layer="94"/>
+</instance>
+<instance part="SB4" gate="G$1" x="-25.4" y="-35.56" smashed="yes" grouprefs="OPEN-CLOSE">
+<attribute name="NAME" x="-30.48" y="-38.1" size="1.778" layer="94"/>
+<attribute name="VALUE" x="-30.48" y="-40.64" size="1.778" layer="94"/>
+</instance>
+<instance part="GND9" gate="1" x="-7.62" y="-17.78" smashed="yes" grouprefs="OPEN-CLOSE">
+<attribute name="VALUE" x="-10.16" y="-20.32" size="1.778" layer="96"/>
 </instance>
 </instances>
@@
 </segment>
 <segment>
-<pinref part="J2" gate="G$1" pin="PIN_2"/>
-<wire x1="66.04" y1="144.78" x2="53.34" y2="144.78" width="0.1524" layer="91" grouprefs="INDOOR_TO_OUTDOOR_CABEL"/>
-<label x="53.34" y="144.78" size="1.778" layer="95" grouprefs="INDOOR_TO_OUTDOOR_CABEL"/>
+<pinref part="SB1" gate="G$1" pin="P$1"/>
+<wire x1="43.18" y1="144.78" x2="27.94" y2="144.78" width="0.1524" layer="91" grouprefs="INDOOR_TO_OUTDOOR_CABEL"/>
+<label x="27.94" y="144.78" size="1.778" layer="95"/>
 </segment>
 </net>
@@
 <wire x1="-172.72" y1="101.6" x2="-172.72" y2="99.06" width="0.1524" layer="91" grouprefs="ESP"/>
 </segment>
+<segment>
+<pinref part="SB4" gate="G$1" pin="P$2"/>
+<pinref part="SB3" gate="G$1" pin="P$2"/>
+<wire x1="-15.24" y1="-35.56" x2="-15.24" y2="-15.24" width="0.1524" layer="91" grouprefs="OPEN-CLOSE"/>
+<pinref part="SB2" gate="G$1" pin="P$2"/>
+<wire x1="-15.24" y1="5.08" x2="-15.24" y2="-15.24" width="0.1524" layer="91" grouprefs="OPEN-CLOSE"/>
+<junction x="-15.24" y="-15.24" grouprefs="OPEN-CLOSE"/>
+<pinref part="GND9" gate="1" pin="GND"/>
+<wire x1="-15.24" y1="-15.24" x2="-7.62" y2="-15.24" width="0.1524" layer="91" grouprefs="OPEN-CLOSE"/>
+</segment>
 </net>
 <net name="GPIO_TS_WINDOW_OPEN" class="0">
 <segment>
-<pinref part="TS1" gate="G$1" pin="P$1"/>
 <wire x1="-35.56" y1="5.08" x2="-71.12" y2="5.08" width="0.1524" layer="91" grouprefs="OPEN-CLOSE"/>
 <label x="-71.12" y="5.08" size="1.778" layer="95" grouprefs="OPEN-CLOSE"/>
+<pinref part="SB2" gate="G$1" pin="P$1"/>
 </segment>
 <segment>
@@
 <net name="GPIO_TS_WINDOW_CLOSE" class="0">
 <segment>
-<pinref part="TS2" gate="G$1" pin="P$1"/>
 <wire x1="-35.56" y1="-15.24" x2="-71.12" y2="-15.24" width="0.1524" layer="91" grouprefs="OPEN-CLOSE"/>
 <label x="-71.12" y="-15.24" size="1.778" layer="95" grouprefs="OPEN-CLOSE"/>
+<pinref part="SB3" gate="G$1" pin="P$1"/>
 </segment>
 <segment>
@@
 <net name="GPIO_TS_WINDOW_AUTO" class="0">
 <segment>
-<pinref part="TS3" gate="G$1" pin="P$1"/>
 <wire x1="-35.56" y1="-35.56" x2="-71.12" y2="-35.56" width="0.1524" layer="91" grouprefs="OPEN-CLOSE"/>
 <label x="-71.12" y="-35.56" size="1.778" layer="95" grouprefs="OPEN-CLOSE"/>
+<pinref part="SB4" gate="G$1" pin="P$1"/>
 </segment>
 <segment>
@@
 </segment>
 </net>
+<net name="N$16" class="0">
+<segment>
+<pinref part="SB1" gate="G$1" pin="P$2"/>
+<pinref part="J2" gate="G$1" pin="PIN_2"/>
+<wire x1="63.5" y1="144.78" x2="66.04" y2="144.78" width="0.1524" layer="91" grouprefs="INDOOR_TO_OUTDOOR_CABEL"/>
+</segment>
+</net>
