File: schematics/main-module/main-module.kicad_sch (KiCad schematic)
At the start: 109 parts, among them J1 Conn_01x02_Socket, J3 Charger, J3 USB_C_Receptacle_USB2.0, J4 Power, J5 Limit Switch, J6 Conn_01x04_Socket, J7 Conn_01x04_Pin, J8 Conn_01x02_Pin, M1 Creality 42-40, Q1 IRF7832PbF, Q14 IRLML0030, Q4 IRF7425PbF, Q7 BC847, SW1 KLS7-TS3601-5.0-180, SW3 Limit Switch, SW4 Limit Switch, SW6 Limit Switch, T1 Transformer_1P_SS, U10 SRX882@315Mhz, U11 FAN3100, U12 FAN3100, U13 TMC2209_Module, U2 CP2102N-Axx-xQFN28, U3 AMS1117-5.0, U4 AMS1117-3.3, U6 SRX882@433Mhz, U7 STX882@433Mhz, U8 ESP32-WROOM-32, U9 TL494

Commit message: 1. board: added protection against high noise in case of endstop is broken. 2. board: added step-up 7.5V -> 15V for charger. 3. firmware - added support for noise protection and some changes in stepper logic
Parts:
- removed C19 (x2): 22 uF, Capacitor_SMD:C_1210_3225Metric, symbol Device:C
- removed C25: 1 nF, Capacitor_SMD:C_0603_1608Metric, symbol Device:C
- removed C25 (x2): 10 uF, Capacitor_SMD:C_0603_1608Metric, symbol Device:C
- removed C25: 500 nF, Capacitor_SMD:C_0603_1608Metric, symbol Device:C
- removed C25 (x2): 100 nF, Capacitor_SMD:C_0603_1608Metric, symbol Device:C
- removed C6: 100 uF, Capacitor_THT:CP_Radial_D6.3mm_P2.50mm, symbol Device:C_Polarized
- removed D2: HER508, Diode_THT:D_DO-201AD_P3.81mm_Vertical_AnodeUp, symbol Device:D
- removed D5: LED, LED_THT:LED_D1.8mm_W3.3mm_H2.4mm, symbol Device:LED
- removed D6: MB10S, Library:MBS, symbol Device:D_Bridge_+-AA
- removed D7: SMAJ5.0CA-TR, Diode_SMD:D_SMA, symbol Diode:ESD9B3.3ST5G
- removed H3: MountingHole, MountingHole:MountingHole_2.2mm_M2, symbol Mechanical:MountingHole
- removed J3: Charger, Connector_JST:JST_XH_B2B-XH-A_1x02_P2.50mm_Vertical, symbol Connector:Conn_01x02_Socket
- removed J4: Power, Connector_JST:JST_XH_B2B-XH-A_1x02_P2.50mm_Vertical, symbol Connector:Conn_01x02_Pin
- removed Q1 (x2): IRF7832PbF, Package_SO:SOIC-8_3.9x4.9mm_P1.27mm, symbol Transistor_FET:IRF7403
- removed Q14: IRLML0030, Package_TO_SOT_SMD:SOT-23, symbol Transistor_FET:IRLML0030
- removed R15 (x4): 1K, Resistor_SMD:R_0805_2012Metric, symbol Device:R
- removed R15 (x3): 10K, Resistor_SMD:R_0805_2012Metric, symbol Device:R
- removed RV2: 1K, Potentiometer_THT:Potentiometer_Runtron_RM-065_Vertical, symbol Device:R_Potentiometer
- removed T1: Transformer_1P_SS, Connector_JST:JST_XH_B5B-XH-A_1x05_P2.50mm_Vertical, symbol Device:Transformer_1P_SS
- removed U11, U12: FAN3100, Package_TO_SOT_SMD:SOT-23-5, symbol My_Library:FAN3100
- removed U9: TL494, Package_SO:SO-16_3.9x9.9mm_P1.27mm, symbol Regulator_Controller:TL494
- added C13, C29, C35, C7: 100 nF, Capacitor_SMD:C_0603_1608Metric, symbol Device:C
- added C16, C17: 22 uF, Capacitor_Tantalum_SMD:CP_EIA-3216-10_Kemet-I_Pad1.58x1.35mm_HandSolder, symbol Device:C_Polarized
- added C18, C33: 10 uF, Capacitor_SMD:C_0603_1608Metric, symbol Device:C
- added C24: 22 uF, Capacitor_SMD:C_1210_3225Metric, symbol Device:C
- added C25, C26, C36: 10 nF, Capacitor_SMD:C_0603_1608Metric, symbol Device:C
- added C32: 220 uF@35V, Capacitor_THT:CP_Radial_D8.0mm_P3.50mm, symbol Device:C_Polarized
- added C8: 47 nF, Capacitor_SMD:C_0603_1608Metric, symbol Device:C
- added D1: SP0503BAHT, Package_TO_SOT_SMD:SOT-143, symbol Power_Protection:SP0503BAHT
- added D3, D5: BAV21WS, Diode_SMD:D_SOD-323F, symbol Device:D
- added D4: SR540, Diode_THT:D_DO-201AD_P3.81mm_Vertical_AnodeUp, symbol Device:D
- added D6: SMAJ26A, Diode_SMD:D_SMA, symbol Diode:SMAJ26A
- added H4: MountingHole, MountingHole:MountingHole_2.2mm_M2, symbol Mechanical:MountingHole
- added J3: Conn_01x02_Pin, symbol Connector:Conn_01x02_Pin
- added J4: Microphone, Connector_JST:JST_XH_B2B-XH-A_1x02_P2.50mm_Vertical, symbol Connector:Conn_01x02_Socket
- added J9: Charger port, Connector_JST:JST_XH_B2B-XH-A_1x02_P2.50mm_Vertical, symbol Connector:Conn_01x02_Socket
- added L1: AMPLF1260, 4.7 uH, Inductor_SMD:L_TaiTech_TMPC1265_13.5x12.5mm, symbol Device:L
- added MK1: Microphone_Condenser, symbol Device:Microphone_Condenser
- added R11, R26: 100K, Resistor_SMD:R_0805_2012Metric, symbol Device:R
- added R15, R20, R6, R8: 10K, Resistor_SMD:R_0805_2012Metric, symbol Device:R
- added R16: 200, Resistor_SMD:R_0805_2012Metric, symbol Device:R
- added R17: 620, Resistor_SMD:R_0805_2012Metric, symbol Device:R
- added R18: 200K, Resistor_SMD:R_0805_2012Metric, symbol Device:R
- added R19, R21: 1K, Resistor_SMD:R_0805_2012Metric, symbol Device:R
- added R25: 0,5, Resistor_SMD:R_2512_6332Metric, symbol Device:R
- added R7: 20K, Resistor_SMD:R_0805_2012Metric, symbol Device:R
- added RV1: RM065, 100K, Potentiometer_THT:Potentiometer_Runtron_RM-065_Vertical, symbol Device:R_Potentiometer
- added TP10: M_EN#, TestPoint:TestPoint_Pad_D1.0mm, symbol Connector:TestPoint
- added TP11: M_STP, TestPoint:TestPoint_Pad_D1.0mm, symbol Connector:TestPoint
- added TP12: M_DIR, TestPoint:TestPoint_Pad_D1.0mm, symbol Connector:TestPoint
- added TP13: VM_EN, TestPoint:TestPoint_Pad_D1.0mm, symbol Connector:TestPoint
- added TP14: CH_FB, TestPoint:TestPoint_Pad_D1.0mm, symbol Connector:TestPoint
- added TP15: CH_CS, TestPoint:TestPoint_Pad_D1.0mm, symbol Connector:TestPoint
- added TP4: NOISE, TestPoint:TestPoint_Pad_D1.0mm, symbol Connector:TestPoint
- added TP7: R315, TestPoint:TestPoint_Pad_D1.0mm, symbol Connector:TestPoint
- added TP8: IC_CE, TestPoint:TestPoint_Pad_D1.0mm, symbol Connector:TestPoint
- added TP9: CH_CE, TestPoint:TestPoint_Pad_D1.0mm, symbol Connector:TestPoint
- added U10: TL331, Package_TO_SOT_SMD:SOT-23-5, symbol Comparator:TL331
- added U12: INA169, Package_TO_SOT_SMD:SOT-23-5, symbol Amplifier_Current:INA169
- added U4: AD8541, Package_TO_SOT_SMD:SOT-23-5, symbol Amplifier_Current:AD8211
- added U8: XL6009, Package_TO_SOT_SMD:TO-263-5_TabPin3, symbol My_Library:XL6009
- J3: symbol Connector:USB_C_Receptacle_USB2.0 -> Connector:USB_C_Receptacle_USB2.0_16P
- TP1: footprint TestPoint:TestPoint_Plated_Hole_D2.0mm -> Library:TestPoint_Plated_Hole_D1.0mm
- TP2: value +5V -> MK_OUT
- TP3: value +3V3 -> NOISE1
- TP5: value GND -> T433; footprint TestPoint:TestPoint_Plated_Hole_D2.0mm -> TestPoint:TestPoint_Pad_D1.0mm
- TP6: value VREF -> R433
- renumbered H4 to H3, J6 to J5, J7 to J6, J5 to J7, SW6 to SW2, SW4 to SW3, SW3 to SW4, U10 to U11, U3 to U2, U13 to U5
Connections:
- net GND1 is gone; now on net FM_OUT_433: TP5.1
- net +3V3: now also C13.1, C17.1, U4.5 (V+); no longer TP3.1
- net +5V: now also C16.1, C29.1, C35.1, C7.1, R15.2, R6.2, R7.2, U10.5 (V+), U12.5 (V+); no longer TP2.1
- net CHARGER_ENABLE: now also C33.2, D5.1 (K), R18.1, TP9.1, U8.2 (EN); no longer U8.8 (IO32)
- net D+: now also D1.4 (K)
- net D-: now also D1.3 (K)
- net FM_IN_5V_315: now also TP7.1
- net FM_IN_5V_433: now also TP6.1
- net GNDA: now also C13.2, C16.2, C17.2, C18.2, C25.1, C26.1, C29.2, C33.1, C35.2, C36.1, C7.2, D1.1 (A), J4.1 (Pin_1), R11.1, R16.1, R26.1, R8.1, RV1.1, U10.2 (V-), U12.2 (GND), U4.2 (GND)
- net GNDPWR: now also C24.1, C32.2, D6.2 (A2), J9.2 (Pin_2), R21.1, U8.1 (GND)
- net M_DIR: now also TP12.1
- net M_ENABLE#: now also TP10.1
- net M_STEP: now also TP11.1
- net VBUS: now also D1.2 (K)
- net VM_ENABLE: now also TP13.1
- net +7.5V_CHARGER_AFTER_FUSE: now reaches F1.2
- net +7.5V_CHARGER_AFTER_FUSE: now also C24.2, L1.2, U8.4 (VIN)
- net NOISE: now reaches U8.7 (IO35)
- net NOISE: now also C18.1, D3.1 (K), R11.2, TP4.1
- new net: D5.2 (A), R17.1, R18.2, U10.4
- new net: C26.2, R15.1, R16.2, U10.1 (-)
- new net: C32.1, D4.1 (K), R19.2, R25.1, U12.3 (+)
- new net: D4.2 (A), L1.1, U8.3 (SW)
- new net: C8.2, R7.1, R8.2, TP2.1, U4.3 (Vin+)
- new net: R19.1, R20.2
- new net: C8.1, J4.2 (Pin_2), R6.1
- new net: D3.2 (A), RV1.3, TP3.1, U4.1 (OUT)
- new net: RV1.2, U4.4 (Vin-)
- new net: D6.1 (A1), J9.1 (Pin_1), R25.2, U12.4 (-)
- new net: J3.1 (Pin_1), MK1.1 (-)
- new net: J3.2 (Pin_2), MK1.2 (+)
- new net CHARGER_CURRENT_SENCE: C25.2, C36.2, R26.2, TP15.1, U10.3 (+), U12.1
- new net CHARGER_FEEDBACK: R20.1, R21.2, TP14.1, U8.5 (FB)
- new net IC_CHARGER_ENABLE: R17.2, TP8.1, U8.8 (IO32)
- no-connect marks 44 -> 43
Other:
- note added: "15V / 1A"
- note added: "Charger port with supply auto-enabling"
- note removed: "-----> WIRE ----->"
- note removed: "Charger module (separated board)"
- moved on the sheet: F1, H3, J3

Commit message: another iteration for outdorr and handle modules
Parts:
- R26: value 100K -> 250K
- RV1: value RM065, 100K -> RM065, 20K
Changed lines of the file:
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@@
 			)
 		)
-		(property "Value" "RM065, 100K"
+		(property "Value" "RM065, 20K"
 			(at 186.69 223.52 0)
 			(effects
@@
 			)
 		)
-		(property "Value" "100K"
+		(property "Value" "250K"
 			(at 480.06 238.7599 0)
 			(effects
