File: schematics/outdoor-module/outdoor-module.kicad_pcb (KiCad board)
At the start: 4 copper layers, 96 x 43 mm, 126 parts, among them J1 2*LiFePo4@18650@1800mAh, 6,4V, J2 USBASP, J4 JST XH B3B, Q1 IRLML5203, Q2 IRLML5203, Q3 IRLML0030, Q4 IRLML0030, Q5 IRLML0030, Q6 IRLML0030, Q7 IRLML0030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

Commit message: changes in second board
Parts:
- moved TP3 8.41 mm to (61.0, 60.4)
- moved C28 7.77 mm to (66.9, 60.1), turned to -90 degrees
- moved C29 7.62 mm to (72.1, 56.6), turned to -90 degrees
- moved U9 6.93 mm to (65.8, 56.8)
- moved U10 4.88 mm to (65.8, 49.4)
- moved RV1 4.35 mm to (69.4, 58.3), turned to 90 degrees
- moved D4 2.21 mm to (69.2, 63.3)
- moved C42 1.00 mm to (74.7, 51.6)
- renumbered C40 to C39, C41 to C40, C42 to C41, C43 to C42, C44 to C43, C45 to C44
Connections:
- RV1 pad 1: GNDA -> +5V
- RV1 pad 3: +5V -> GNDA
Routing:
- net +5V: track 230.6 -> 238.4 mm, vias 10 -> 11
- net +1V8: track 29.1 -> 34.6 mm
- net Net-(U10-Vin-): track 3.04 -> 7.29 mm
- net /NOISE: track 28.9 -> 31.7 mm
- net /NOISE_ALARM: track 25.8 -> 23.4 mm
- net Net-(U9-Vin-): track 9.71 -> 7.44 mm
- net Net-(D4-A): track 6.03 -> 8.03 mm
- net Net-(U10-Vin+): track 8.67 -> 7.11 mm
- net GNDA: track 161.3 -> 160.3 mm

Commit message: Project prepared to order
Parts:
- moved C3 0.37 mm to (83.0, 80.2)
- moved R29 0.32 mm to (118.8, 78.2)
- moved C8 0.18 mm to (96.6, 78.2)
- moved R2 0.16 mm to (73.0, 65.9)
- moved C23 0.14 mm to (72.2, 41.8), turned to -90 degrees
- moved Q1 0.13 mm to (69.8, 69.6)
- moved C32 0.10 mm to (126.3, 70.9)
- moved C7 0.10 mm to (90.0, 80.2)
- moved R1 0.05 mm to (73.0, 69.6)
Connections:
- TP2 pad 1: GNDPWR -> GNDA
Routing:
- net GNDPWR: track 196.6 -> 183.4 mm
- net GNDA: track 160.3 -> 167.5 mm
- net Net-(U6-EN): track 5.42 -> 4.80 mm
Other:
- board text added: "0,0000 mm / 0,0000 mm"
- board text added: "0,2000 mm"
- board text added: "1,6000 mm"
- board text added: "4"
- board text added: "96,0000 mm x 43,0000 mm"
- board text added: "ACW-outdoor-v1.0.1"
- board text added: "None"
- board text added: "Габариты платы:"
- board text added: "Количество слоёв меди:"
- board text added: "Контроль импеданса:"
- board text added: "Краевой соединитель:"
- board text added: "Метал. торцы:"
- board text added: "Мин. дорожка/зазор:"
- board text added: "Мин. сверло:"
- board text added: "Нет"
- board text added: "Периферийные полу-отверстия:"
- board text added: "Покрытие меди:"
- board text added: "Толщина платы:"
- board text added: "ХАРАКТЕРИСТИКИ ПЛАТЫ"
- board text removed: "ACW - outdoor v1.0"

Commit message: another iteration for outdorr and handle modules
Parts:
- removed C43: 10 uF, Capacitor_SMD:C_0603_1608Metric
- removed D2: 15MQ030NPBF, Diode_SMD:D_SMA
- removed J4: JST XH B3B, Connector_JST:JST_XH_B3B-XH-A_1x03_P2.50mm_Vertical
- removed JP1: AC Detect, Jumper:SolderJumper-2_P1.3mm_Open_TrianglePad1.0x1.5mm
- removed R22: 6R8, Resistor_SMD:R_0805_2012Metric
- removed TP8: CHG SUPPLY, TestPoint:TestPoint_Pad_D1.0mm
- added C45: 100 nF, Capacitor_SMD:C_0603_1608Metric, B.Cu at (124.6, 76.0)
- added J3: Charger, Connector_JST:JST_XH_B2B-XH-A_1x02_P2.50mm_Vertical, F.Cu at (133.1, 45.6)
- added NT2: NetTie_2, NetTie:NetTie-2_SMD_Pad0.5mm, F.Cu at (116.4, 75.0)
- added NT3: NetTie_2, NetTie:NetTie-2_SMD_Pad0.5mm, F.Cu at (114.7, 75.0)
- added TP11: ACDRV, TestPoint:TestPoint_Pad_D1.0mm, F.Cu at (118.6, 57.4)
- added TP12: ACOK, TestPoint:TestPoint_Pad_D1.0mm, F.Cu at (115.2, 58.2)
- added U12: INA219, Package_SO:SOIC-8_3.9x4.9mm_P1.27mm, B.Cu at (124.8, 79.6)
- C24, C27, C30, R21: moved to F.Cu
- C36: value 10 nF -> 4.7 uF
- D6: value ES2J -> SMAJ26A; footprint Diode_SMD:D_SMB -> Diode_SMD:D_SMA; moved to B.Cu
- D7, NT1: moved to B.Cu
- R20: value 10K -> 2K2; moved to B.Cu
- R29: value 100K -> 10
- R30: value 4K7 -> 10
- TP1: value VBAT -> CHG SUPPLY
- TP2: footprint TestPoint:TestPoint_Plated_Hole_D2.0mm -> Library:TestPoint_Plated_Hole_D1.0mm
- TP9: value ILIM -> ACDET
- moved Q7 35.1 mm to (134.2, 73.0), turned to 90 degrees
- moved R20 34.2 mm to (135.8, 44.4), turned to -90 degrees
- moved R17 33.2 mm to (135.2, 76.9), turned to -90 degrees
- moved R18 30.8 mm to (133.2, 76.9), turned to -90 degrees
- moved TP1 26.7 mm to (111.0, 49.4)
- moved H2 22.7 mm to (107.0, 47.5)
- moved C36 22.3 mm to (112.8, 43.6)
- moved TP9 21.1 mm to (113.0, 60.8)
- moved NT1 18.1 mm to (102.8, 81.8)
- moved C7 17.3 mm to (107.2, 78.0), turned to -90 degrees
- moved C8 17.1 mm to (113.6, 79.6), turned to -90 degrees
- moved C11 17.0 mm to (111.0, 79.6), turned to 90 degrees
- moved C10 17.0 mm to (109.2, 79.6), turned to -90 degrees
- moved C3 15.7 mm to (98.6, 78.0), turned to -90 degrees
- moved H1 11.5 mm to (112.0, 73.5)
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Connections:
- net /CHARGER_PHASE renamed Net-(Q5-S)
- C10 pad 1: /VBAT_BEFORE_FUSE -> /VBAT
- C11 pad 2: /VBAT_BEFORE_FUSE -> /VBAT
- C14 pad 1: Net-(D2-K) -> /VSYS
- C26 pad 1: Net-(U8-REGN) -> Net-(U8-ILIM)
- C3 pad 1: /VBAT_BEFORE_FUSE -> /VBAT
- C32 pad 1: Net-(C32-Pad1) -> Net-(U8-BTST)
- C36 pad 1: Net-(D6-A) -> /CHARGER_SUPPLY
- C36 pad 2: Net-(D7-A) -> GNDPWR
- C7 pad 1: /VBAT_BEFORE_FUSE -> /VBAT
- C8 pad 1: /VBAT_BEFORE_FUSE -> /VBAT
- D6 pad 1: Net-(D6-K) -> Net-(D6-A1)
- D6 pad 2: Net-(D6-A) -> GNDPWR
- D7 pad 1: Net-(D6-K) -> Net-(D7-K)
- D7 pad 2: Net-(D7-A) -> Net-(D6-A1)
- F1 pad 1: /VBAT_BEFORE_FUSE -> Net-(J1-Pin_2)
- F2 pad 1: Net-(D6-K) -> Net-(D7-K)
- J1 pad 2: /VBAT_BEFORE_FUSE -> Net-(J1-Pin_2)
- R20 pad 1: Net-(U8-TB_STAT#) -> Net-(D6-A1)
- R20 pad 2: +5V -> GNDPWR
- R24 pad 2: /CHARGER_BATSRC -> Net-(U8-SRP)
- R28 pad 1: /VBAT -> /CHARGER_SRN
- R28 pad 2: /CHARGER_SRN -> Net-(U8-SRN)
- R29 pad 1: +5V -> Net-(U12-VIN_+)
- R29 pad 2: /CHARGER_ILIM -> /CHARGER_SRP
- R30 pad 1: /CHARGER_ILIM -> /CHARGER_SRN
- R30 pad 2: GNDA -> Net-(U12-VIN_-)
- R8 pad 2: Net-(JP1-A) -> Net-(U8-ACDET)
- R9 pad 1: Net-(JP1-A) -> Net-(U8-ACDET)
- TP1 pad 1: /VBAT -> /CHARGER_SUPPLY
- TP9 pad 1: /CHARGER_ILIM -> Net-(U8-ACDET)
- U3 pad 3: Net-(D2-K) -> /VSYS
- U8 pad 13: GNDA -> GNDPWR
- U8 pad 16: Net-(U8-TB_STAT#) -> unconnected-(U8-TB_STAT#-Pad16)
- U8 pad 19: /CHARGER_SRN -> Net-(U8-SRN)
- U8 pad 20: /CHARGER_SRP -> Net-(U8-SRP)
- U8 pad 21: /CHARGER_ILIM -> Net-(U8-ILIM)
- U8 pad 24: Net-(U8-REGN) -> Net-(U8-ILIM)
- U8 pad 25: /CHARGER_BOOST -> Net-(U8-BTST)
- U8 pad 6: Net-(JP1-B) -> Net-(U8-ACDET)
Routing:
- net GNDPWR: track 183.4 -> 130.3 mm
- net /SDA: track 63.4 -> 92.1 mm, vias 3 -> 4
- net /SCL: track 63.8 -> 89.5 mm, vias 3 -> 4
- net /VBAT_BEFORE_FUSE: track 25.4 -> 0.00 mm
- net /CHARGER_BATSRC: track 48.5 -> 25.5 mm, vias 2 -> 3
- net /VBAT: track 22.2 -> 43.1 mm, vias 2 -> 1
- net /CHARGER_SUPPLY: track 62.0 -> 43.5 mm
- net Net-(U8-ACDET): track 0.00 -> 16.0 mm
- net /VSYS: track 83.3 -> 98.0 mm, vias 3 -> 2
- net Net-(JP1-B): track 13.5 -> 0.00 mm
- net /CHARGER_ILIM: track 12.8 -> 0.00 mm
- net Net-(D6-A1): track 0.00 -> 11.7 mm
- net Net-(D6-K): track 10.2 -> 0.00 mm
- net Net-(D2-K): track 8.65 -> 0.00 mm
- net Net-(D7-A): track 8.24 -> 0.00 mm
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Other:
- board text added: "ACW-outdoor-v1.1.0"
- board text removed: "ACW-outdoor-v1.0.1"
