File: schematics/outdoor-module/outdoor-module.kicad_sch (KiCad schematic)
At the start: 122 parts, among them J1 2*LiFePo4@18650@1800mAh, 6,4V, J3 FS1000A@315Mhz, J4 BME280, J4 USBASP, J5 JST XH B3B, J6 JST XH B3B, Q10 IRLML5203, Q3 IRLML0030, U1 PCA9306, U12 ATmega328-A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

Commit message: Second board
Parts:
- removed C19, C29: 22 uF, Capacitor_SMD:C_1210_3225Metric, symbol Device:C
- removed J3: FS1000A@315Mhz, symbol Connector:Conn_01x03_Socket
- removed J4: BME280, symbol Connector:Conn_01x04_Socket
- added C26 (x2): 100 nF, Capacitor_SMD:C_0603_1608Metric, symbol Device:C
- added H1, H2, H3, H4, H5: MountingHole, MountingHole:MountingHole_2.2mm_M2, symbol Mechanical:MountingHole
- added TP7: MK_OUT, TestPoint:TestPoint_Pad_D1.0mm, symbol Connector:TestPoint
- added TP7: NOISE, TestPoint:TestPoint_Pad_D1.0mm, symbol Connector:TestPoint
- added U2: STX882@315MHz, Library:STX882_Vertical, symbol My_Library:STX882
- added U7: BME280, Package_LGA:Bosch_LGA-8_2.5x2.5mm_P0.65mm_ClockwisePinNumbering, symbol Sensor:BME280
- C26: value 10 uF -> 100 nF
- F2: value 2A -> 3A
- MK1: footprint (none) -> Library:SMD03722C4
- R15: value 7K -> 4K7
- R2, R3: value 3.3K -> 4K7
- R28: value 10K -> 4K7
- renumbered J6 to J3, J5 to J4, U8 to U10, U4 to U5, U7 to U9
Connections:
- net +3V3: now also C26.1, U7.2 (CSB), U7.6 (VDDIO), U7.8 (VDD); no longer R15.1
- net +5V: now also C26.1, C29.1, R15.1, U3.3 (VI), U5.3 (VI), C26.1, U2.3 (VCC)
- net CHARGER_DONE#: now also U12.2 (PD4); no longer U12.12 (PB0)
- net CHARGER_IN_PROGRESS#: now also U12.1 (PD3); no longer U12.13 (PB1)
- net FM_OUT: now also U12.9 (PD5), U2.2 (DATA); no longer U12.14 (PB2)
- net GNDA: now also C26.2, C26.2, C26.2, U2.4 (GND), U7.1 (GND), U7.5 (SDO), U7.7 (GND)
- net GNDPWR: no longer C26.2
- net NOISE: now also U12.25 (PC2), TP7.1; no longer U12.23 (PC0)
- net SCK: no longer C27.1, U12.7 (XTAL1/PB6), X1.2
- net at C26.2, R3.1, R3.2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: now also TP7.1
- net BME_SCL renamed SCL_3V3
- net SCL_3V3: now also U7.4 (SCK)
- net BME_SDA renamed SDA_3V3
- net SDA_3V3: now also U7.3 (SDI)
- new net: C27.1, U12.7 (XTAL1/PB6), X1.2
- new net: C29.1, D6.1 (K), U3.3 (VI)
Other:
- note added: "0,05A"
- note added: "0,2A"
- note removed: "0,1A"
- note removed: "0,5A"
- moved on the sheet: C26, TP6

Commit message: changes in second board
Connections:
- net +5V: now also RV4.1; no longer RV4.3
- net GNDA: now also RV4.3; no longer RV4.1
Other:
- moved on the sheet: RV4

Commit message: Project prepared to order
Connections:
- net GNDA: now also TP2.1
- net GNDPWR: no longer TP2.1
Changed lines of the file:
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@@
   )
   (symbol (lib_id "My_Library:BQ24780S") (at 368.3 212.09 0) (unit 1)
-    (in_bom yes) (on_board yes) (dnp no) (fields_autoplaced)
-    (property "Reference" "U5" (at 371.7641 184.15 0)
+    (in_bom yes) (on_board yes) (dnp no)
+    (property "Reference" "U5" (at 377.19 181.61 0)
       (effects (font (size 1.27 1.27)) (justify left))
     )
-    (property "Value" "BQ24780S" (at 359.41 193.04 0)
+    (property "Value" "BQ24780S" (at 382.27 184.15 0)
       (effects (font (size 1.27 1.27)))
     )
@@
     )
   )
+  (symbol (lib_id "power:GNDA") (at 67.31 67.31 0) (unit 1)
+    (in_bom yes) (on_board yes) (dnp no)
+    (property "Reference" "#PWR015" (at 67.31 73.66 0)
+      (effects (font (size 1.27 1.27)) hide)
+    )
+    (property "Value" "GNDA" (at 67.31 72.39 0)
+      (effects (font (size 1.27 1.27)))
+    )
+    (property "Footprint" "" (at 67.31 67.31 0)
+      (effects (font (size 1.27 1.27)) hide)
+    )
+    (property "Datasheet" "" (at 67.31 67.31 0)
+      (effects (font (size 1.27 1.27)) hide)
+    )
+    (pin "1")
+    (instances
+      (project "handle-module"
+        (path "/5a1662b2-39be-45fc-af40-ee8b9104876f"
+          (reference "#PWR015") (unit 1)
+        )
+      )
+      (project "outdoor-module"
+        (path "/f407c3fc-0a96-48ff-b74a-a4fbb61aa182"
+          (reference "#PWR09") (unit 1)
+        )
+      )
+    )
+  )
   (symbol (lib_id "power:GNDA") (at 426.72 379.73 0) (unit 1)
     (in_bom yes) (on_board yes) (dnp no)
@@
         )
       )
-    )
-  )
-  (symbol (lib_id "power:GNDPWR") (at 67.31 67.31 0) (unit 1)
-    (in_bom yes) (on_board yes) (dnp no)
-    (property "Reference" "#PWR014" (at 67.31 72.39 0)
-      (effects (font (size 1.27 1.27)) hide)
-    )
-    (property "Value" "GNDPWR" (at 67.183 71.12 0)
-      (effects (font (size 1.27 1.27)))
-    )
-    (property "Footprint" "" (at 67.31 68.58 0)
-      (effects (font (size 1.27 1.27)) hide)
-    )
-    (property "Datasheet" "" (at 67.31 68.58 0)
-      (effects (font (size 1.27 1.27)) hide)
-    )
-    (pin "1")
-    (instances
-      (project "handle-module"
-        (path "/5a1662b2-39be-45fc-af40-ee8b9104876f"
-          (reference "#PWR014") (unit 1)
-        )
-      )
-      (project "outdoor-module"
-        (path "/f407c3fc-0a96-48ff-b74a-a4fbb61aa182"
-          (reference "#PWR09") (unit 1)
-        )
-      )

Commit message: another iteration for outdorr and handle modules
Parts:
- removed C26: 10 uF, Capacitor_SMD:C_0603_1608Metric, symbol Device:C
- removed C26: 10 nF, Capacitor_SMD:C_0603_1608Metric, symbol Device:C
- removed D10, D9: ES2J, Diode_SMD:D_SMB, symbol Device:D
- removed D6: 15MQ030NPBF, Diode_SMD:D_SMA, symbol Device:D
- removed J3: JST XH B3B, symbol Connector:Conn_01x03_Pin
- removed J4: JST XH B3B, Connector_JST:JST_XH_B3B-XH-A_1x03_P2.50mm_Vertical, symbol Connector:Conn_01x03_Socket
- removed JP1: AC Detect, Jumper:SolderJumper-2_P1.3mm_Open_TrianglePad1.0x1.5mm, symbol Jumper:SolderJumper_2_Open
- removed L1, L2: ?, symbol Device:L
- removed R15: 6R8, Resistor_SMD:R_0805_2012Metric, symbol Device:R
- removed R15: 10K, Resistor_SMD:R_0805_2012Metric, symbol Device:R
- removed R15: 4K7, Resistor_SMD:R_0805_2012Metric, symbol Device:R
- removed R15: 100K, Resistor_SMD:R_0805_2012Metric, symbol Device:R
- removed RV1: JVR-05N180M, Varistor:RV_Disc_D7mm_W4.5mm_P5mm, symbol Device:Varistor
- removed TP7: CHG SUPPLY, TestPoint:TestPoint_Pad_D1.0mm, symbol Connector:TestPoint
- removed TP8: ILIM, TestPoint:TestPoint_Pad_D1.0mm, symbol Connector:TestPoint
- added C36: 4.7 uF, Capacitor_SMD:C_0603_1608Metric, symbol Device:C
- added C45: 100 nF, Capacitor_SMD:C_0603_1608Metric, symbol Device:C
- added D6: SMAJ26A, Diode_SMD:D_SMA, symbol Diode:SMAJ26A
- added D7: ES2J, Diode_SMD:D_SMB, symbol Device:D
- added J3: Charger, Connector_JST:JST_XH_B2B-XH-A_1x02_P2.50mm_Vertical, symbol Connector:Conn_01x02_Socket
- added NT2, NT3: NetTie_2, NetTie:NetTie-2_SMD_Pad0.5mm, symbol Device:NetTie_2
- added R20: 2K2, Resistor_SMD:R_0805_2012Metric, symbol Device:R
- added R29, R30: 10, Resistor_SMD:R_0805_2012Metric, symbol Device:R
- added RV2: JVR-05N180M, Varistor:RV_Disc_D7mm_W4.5mm_P5mm, symbol Device:Varistor
- added TP11: ACDRV, TestPoint:TestPoint_Pad_D1.0mm, symbol Connector:TestPoint
- added TP12: ACOK, TestPoint:TestPoint_Pad_D1.0mm, symbol Connector:TestPoint
- added TP9: ACDET, TestPoint:TestPoint_Pad_D1.0mm, symbol Connector:TestPoint
- added U12: INA219, Package_SO:SOIC-8_3.9x4.9mm_P1.27mm, symbol My_Library:INA219
- TP1: value VBAT -> CHG SUPPLY
- TP2: footprint TestPoint:TestPoint_Plated_Hole_D2.0mm -> Library:TestPoint_Plated_Hole_D1.0mm
Connections:
- net CHARGER_BOOST is gone; now on an unnamed net: U5.25 (BTST)
- net CHARGER_ILIM is gone; now on an unnamed net: U5.21 (ILIM)
- net +5V: now also C45.1, U12.5 (VCC)
- net CHARGER_BATSRC: now also NT2.2; no longer R15.2
- net CHARGER_SRN: now also R15.1, NT3.1, R30.1; no longer R15.2, U5.19 (SRN)
- net CHARGER_SRP: now also NT2.1, R29.2; no longer U5.20 (SRP)
- net CHARGER_SUPPLY: now also TP1.1, C36.1, RV2.1
- net GNDA: now also C45.2, U12.6 (GND); no longer U5.13 (CMPIN)
- net GNDPWR: now also U5.13 (CMPIN), C36.2, D6.2 (A2), J3.1 (Pin_1), R20.2, RV2.2
- net SCL: now also U12.4 (SCL)
- net SDA: now also U12.1 (A1), U12.2 (A0), U12.3 (SDA)
- net VBAT: now also C18.2, C26.1, C29.1, C5.1, C6.1, NT3.2; no longer R15.1, TP1.1
- net VSYS: now also C29.1, U3.3 (VI)
- net at C26.2, C26.2, Q3.1 (G)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: now also TP11.1
- net at F2.1: now also D7.1 (K)
- net at R15.1, U5.5 (ACOK): now also TP12.1
- net at U5.6 (ACDET): now also R15.1, R15.2, TP9.1
- net CHARGER_PHASE: no longer names the net of C26.2, L3.1, Q3.2 (S), Q3.3 (D), U5.27 (PHASE)
- removed net VBAT_BEFORE_FUSE: C18.2, C26.1, C29.1, C5.1, C6.1, F1.1, J1.2 (Pin_2)
- new net: R29.1, U12.8 (VIN_+)
- new net: F1.1, J1.2 (Pin_2)
- new net: R15.2, U5.19 (SRN)
- new net: R15.2, U5.20 (SRP)
- new net: D6.1 (A1), D7.2 (A), J3.2 (Pin_2), R20.1
- new net: R30.2, U12.7 (VIN_-)
- no-connect marks 17 -> 18
Other:
- note added: "I2C address 0x09"
- note added: "I2C address 0x4A"
- note added: "I2C address: 0x76"
- moved on the sheet: C26, C29, F1, R15
