File: schematics/handle-module/handle-module.kicad_sch (KiCad schematic)
At the start: 108 parts, among them J1 2*LiFePo4@18650@1800mAh, 6,4V, J2 Charger, J4 USBASP, Q10 IRLML5203, Q3 IRLML0030, Q5 IRLML0030, Q6 IRLML5203, SW1 KLS7-TS3601-5.0-180, SW2 KLS7-TS3601-5.0-180, U1 STX882@443MHz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

Commit message: another iteration for outdorr and handle modules
Parts:
- removed TP1: VBAT, TestPoint:TestPoint_Pad_D1.0mm, symbol Connector:TestPoint
- added C33: 100 nF, Capacitor_SMD:C_0603_1608Metric, symbol Device:C
- added JP1: PROCHOT#_EN, Jumper:SolderJumper-2_P1.3mm_Open_TrianglePad1.0x1.5mm, symbol Jumper:SolderJumper_2_Open
- added NT2, NT3: NetTie_2, NetTie:NetTie-2_SMD_Pad0.5mm, symbol Device:NetTie_2
- added R28, R29: 10, Resistor_SMD:R_0805_2012Metric, symbol Device:R
- added U7: INA219, Package_SO:SOIC-8_3.9x4.9mm_P1.27mm, symbol My_Library:INA219
- R23: value 500 -> 2K2
Connections:
- net +5V: now also C33.1, U7.5 (VCC)
- net CHARGER_BATSRC: now also NT2.2; no longer R15.2
- net CHARGER_SRN: now also R15.1, NT3.1, R28.1; no longer R15.2, U5.19 (SRN)
- net CHARGER_SRP: now also R15.2, NT2.1, R29.2; no longer R15.1, U5.20 (SRP)
- net CHARGER_SUPPLY: now also D7.1 (A1)
- net GNDA: now also TP2.1, C33.2, U7.6 (GND); no longer U5.21 (ILIM)
- net GNDPWR: now also U5.13 (CMPIN); no longer TP2.1
- net SCL: now also U7.4 (SCL)
- net SDA: now also U7.1 (A1), U7.2 (A0), U7.3 (SDA)
- net VBAT: now also C18.2, C26.1, C29.1, C5.1, C6.1, NT3.2; no longer R15.1
- net at D9.2 (A), J2.2 (Pin_2), R23.1: no longer D7.1 (A1)
- net at U5.10 (PROCHOT#): now also JP1.1 (A)
- net at C26.1, U5.24 (REGN): now also U5.21 (ILIM)
- net PROCHOT#: now reaches Q5.3 (D), Q6.1 (G), R9.2
- net PROCHOT#: now also JP1.2 (B)
- removed net VBAT_BEFORE_FUSE: C18.2, C26.1, C29.1, C5.1, C6.1, F1.1, J1.2 (Pin_2)
- new net: R15.1, U5.20 (SRP)
- new net: R28.2, U7.8 (VIN_+)
- new net: F1.1, J1.2 (Pin_2)
- new net: R29.1, U7.7 (VIN_-)
- new net: R15.2, U5.19 (SRN)
- no-connect marks 18 -> 16
Other:
- note added: "I2C address 0x09"
- note added: "I2C address 0x4A"
- moved on the sheet: C26, D7, D9, F1, F2, R15, R23, TP6

Commit message: handle module & main module almost done
Parts:
- D9: value ES2J -> SS34BF
Changed lines of the file:
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@@
 		)
 	)
+	(text_box "SS34BF"
+		(exclude_from_sim no)
+		(at 416.56 21.59 0)
+		(size 10.16 5.08)
+		(stroke
+			(width 0)
+			(type default)
+		)
+		(fill
+			(type none)
+		)
+		(effects
+			(font
+				(size 1.27 1.27)
+			)
+			(justify left top)
+		)
+	)
 	(text "AVG 1A\nMAX 2A"
 		(exclude_from_sim no)
@@
 		(instances
 			(project "supply"
-				(path "/1e139717-fcd1-4008-a6ea-4c993845e928/bcabd54f-a555-4409-9a4f-89c20a3d7682"
-					(reference "C18")
-					(unit 1)
-				)
 				(path "/1e139717-fcd1-4008-a6ea-4c993845e928/4671650e-ec71-47e3-a051-fc2ad6d25f63"
 					(reference "C50")
 					(unit 1)
 				)
+				(path "/1e139717-fcd1-4008-a6ea-4c993845e928/bcabd54f-a555-4409-9a4f-89c20a3d7682"
+					(reference "C18")
+					(unit 1)
+				)
 			)
 			(project "handle-module"
@@
 			)
 			(project "supply"
-				(path "/1e139717-fcd1-4008-a6ea-4c993845e928/ce2ff71a-422a-4b17-921a-2433d38ec044"
-					(reference "Q9")
-					(unit 1)
-				)
 				(path "/1e139717-fcd1-4008-a6ea-4c993845e928/39d9543b-2a42-4758-87e9-56ce3e85ea36"
 					(reference "Q11")
 					(unit 1)
 				)
+				(path "/1e139717-fcd1-4008-a6ea-4c993845e928/ce2ff71a-422a-4b17-921a-2433d38ec044"
+					(reference "Q9")
+					(unit 1)
+				)
 			)
 			(project "handle-module"
@@
 		(instances
 			(project "supply"
-				(path "/1e139717-fcd1-4008-a6ea-4c993845e928/ce2ff71a-422a-4b17-921a-2433d38ec044"
-					(reference "R54")
-					(unit 1)
-				)
 				(path "/1e139717-fcd1-4008-a6ea-4c993845e928/39d9543b-2a42-4758-87e9-56ce3e85ea36"
 					(reference "R55")
 					(unit 1)
 				)
+				(path "/1e139717-fcd1-4008-a6ea-4c993845e928/ce2ff71a-422a-4b17-921a-2433d38ec044"
+					(reference "R54")
+					(unit 1)
+				)
 			)
 			(project "handle-module"
@@
 		(instances
 			(project "supply"
-				(path "/1e139717-fcd1-4008-a6ea-4c993845e928/bcabd54f-a555-4409-9a4f-89c20a3d7682"
-					(reference "C18")
-					(unit 1)
-				)
 				(path "/1e139717-fcd1-4008-a6ea-4c993845e928/4671650e-ec71-47e3-a051-fc2ad6d25f63"
 					(reference "C50")
 					(unit 1)
 				)
+				(path "/1e139717-fcd1-4008-a6ea-4c993845e928/bcabd54f-a555-4409-9a4f-89c20a3d7682"
+					(reference "C18")
+					(unit 1)
+				)
 			)
 			(project "handle-module"
@@
 			)
 			(project "supply"
-				(path "/1e139717-fcd1-4008-a6ea-4c993845e928/ce2ff71a-422a-4b17-921a-2433d38ec044"
-					(reference "Q9")
-					(unit 1)
-				)
 				(path "/1e139717-fcd1-4008-a6ea-4c993845e928/39d9543b-2a42-4758-87e9-56ce3e85ea36"
 					(reference "Q11")
 					(unit 1)
 				)
+				(path "/1e139717-fcd1-4008-a6ea-4c993845e928/ce2ff71a-422a-4b17-921a-2433d38ec044"
+					(reference "Q9")
+					(unit 1)
+				)
 			)
 			(project "handle-module"
@@
 		(instances
 			(project "supply"
-				(path "/1e139717-fcd1-4008-a6ea-4c993845e928/bcabd54f-a555-4409-9a4f-89c20a3d7682"
-					(reference "C18")
-					(unit 1)
-				)
 				(path "/1e139717-fcd1-4008-a6ea-4c993845e928/4671650e-ec71-47e3-a051-fc2ad6d25f63"
 					(reference "C50")
 					(unit 1)
 				)
+				(path "/1e139717-fcd1-4008-a6ea-4c993845e928/bcabd54f-a555-4409-9a4f-89c20a3d7682"
+					(reference "C18")
+					(unit 1)
+				)
 			)
 			(project "handle-module"
@@
 		(instances
 			(project "supply"
-				(path "/1e139717-fcd1-4008-a6ea-4c993845e928/ce2ff71a-422a-4b17-921a-2433d38ec044"
-					(reference "R54")
-					(unit 1)
-				)
 				(path "/1e139717-fcd1-4008-a6ea-4c993845e928/39d9543b-2a42-4758-87e9-56ce3e85ea36"
 					(reference "R55")
 					(unit 1)
 				)
+				(path "/1e139717-fcd1-4008-a6ea-4c993845e928/ce2ff71a-422a-4b17-921a-2433d38ec044"
+					(reference "R54")
+					(unit 1)
+				)
 			)
 			(project "handle-module"
@@
 			)
 		)
-		(property "Value" "ES2J"
+		(property "Value" "SS34BF"
 			(at 420.37 30.48 0)
 			(effects

Commit message: prepare to change ADC working mode to continuus
Parts:
- renumbered C18 to C50, R54 to R55
Changed lines of the file:
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@@
 		)
 	)
+	(text_box "change to 60K"
+		(exclude_from_sim no)
+		(at 283.21 205.74 0)
+		(size 21.59 3.81)
+		(stroke
+			(width 0)
+			(type default)
+		)
+		(fill
+			(type none)
+		)
+		(effects
+			(font
+				(size 1.27 1.27)
+			)
+			(justify left top)
+		)
+	)
 	(text_box "SS34BF"
 		(exclude_from_sim no)
@@
 		(on_board yes)
 		(dnp no)
-		(property "Reference" "C18"
+		(property "Reference" "C50"
 			(at 165.1 46.99 0)
 			(effects
@@
 		(dnp no)
 		(fields_autoplaced yes)
-		(property "Reference" "R54"
+		(property "Reference" "R55"
 			(at 59.69 367.03 0)
 			(effects
@@
 		(on_board yes)
 		(dnp no)
-		(property "Reference" "C18"
+		(property "Reference" "C50"
 			(at 82.55 133.35 0)
 			(effects
@@
 		(on_board yes)
 		(dnp no)
-		(property "Reference" "C18"
+		(property "Reference" "C50"
 			(at 81.28 189.23 0)
 			(effects
@@
 		(dnp no)
 		(fields_autoplaced yes)
-		(property "Reference" "R54"
+		(property "Reference" "R55"
 			(at 60.96 337.82 0)
 			(effects
